File: PCBcam/PCBcam.kicad_pcb (KiCad board)
At the start: 2 copper layers, 53.8 x 27.4 mm, 11 parts, among them J1 Rx/Tx, J2 Conn_01x02, J3 5V-Gnd

Commit message: chore(PCB): PCB layout added
Parts:
- moved REF** 6.10 mm to (147.3, 96.5)
Routing:
- net gnd: vias 0 -> 3
Other:
- board size 53.8 x 27.4 mm -> 53.8 x 34 mm
Changed lines of the file:
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@@
   (general
     (thickness 1.6)
-    (drawings 16)
-    (tracks 39)
+    (drawings 17)
+    (tracks 42)
     (zones 0)
     (modules 11)
@@
   )
   (module MountingHole:MountingHole_2.5mm_Pad (layer F.Cu)
-    (at 147.32 90.424)
+    (at 147.32 96.52)
     (descr "Mounting Hole 2.5mm")
     (tags "mounting hole 2.5mm")
@@
     )
   )
-  (gr_line (start 142.748 94.996) (end 150.368 94.996) (layer Edge.Cuts) (width 0.05))
+  (gr_line (start 196.596 101.6) (end 196.596 94.996) (layer Edge.Cuts) (width 0.05))
+  (gr_line (start 142.748 101.6) (end 196.596 101.6) (layer Edge.Cuts) (width 0.05))
+  (gr_line (start 142.748 94.996) (end 142.748 101.6) (layer Edge.Cuts) (width 0.05))
   (gr_line (start 142.748 67.564) (end 142.748 94.996) (layer Edge.Cuts) (width 0.05))
   (gr_line (start 150.368 67.564) (end 142.748 67.564) (layer Edge.Cuts) (width 0.05))
@@
     (arrow2b (pts (xy 142.748 63.5) (xy 143.874504 62.913579)))
   )
-  (gr_line (start 150.368 94.996) (end 196.596 94.996) (layer Edge.Cuts) (width 0.05))
   (gr_line (start 196.596 67.564) (end 150.368 67.564) (layer Edge.Cuts) (width 0.05))
   (segment (start 185.4454 89.3826) (end 184.912 89.916) (width 0.5) (layer B.Cu) (net 9))
@@
   (segment (start 186.436 80.772) (end 184.912 82.296) (width 0.5) (layer F.Cu) (net 11))
   (segment (start 194.056 80.772) (end 186.436 80.772) (width 0.5) (layer F.Cu) (net 11))
+  (via (at 154.432 88.9) (size 0.8) (drill 0.4) (layers F.Cu B.Cu) (net 11))
+  (via (at 192.532 97.536) (size 0.8) (drill 0.4) (layers F.Cu B.Cu) (net 11))
+  (via (at 173.228 96.012) (size 0.8) (drill 0.4) (layers F.Cu B.Cu) (net 11))
   (segment (start 186.436 78.232) (end 184.912 79.756) (width 0.5) (layer F.Cu) (net 12))
   (segment (start 194.056 78.232) (end 186.436 78.232) (width 0.5) (layer F.Cu) (net 12))
@@
     (polygon
       (pts
-        (xy 196.596 94.996) (xy 142.748 94.996) (xy 142.748 67.564) (xy 196.596 67.564)
+        (xy 196.596 101.6) (xy 142.748 101.6) (xy 142.748 67.564) (xy 196.596 67.564)
       )
     )
@@
     (polygon
       (pts
-        (xy 196.596 94.996) (xy 142.748 94.996) (xy 142.748 67.564) (xy 196.596 67.564)
+        (xy 196.596 101.6) (xy 142.748 101.6) (xy 142.748 67.564) (xy 196.596 67.564)
       )
     )
